File: hardware/goose60rev2/connector.kicad_sch (KiCad schematic)
At the start: 14 parts, among them J1 USB_C_Receptacle_USB2.0_14P, J3 Conn_01x04_Socket, J4 Conn_01x04_Socket, J5 Conn_01x12_Socket, U2 TXS0108EPW, U6 USBLC6-2SC6

Commit message: update sch design
Parts:
- removed J5: Conn_01x12_Socket, symbol Connector:Conn_01x12_Socket
- added D2, D3: 3.6V, symbol Device:D_Zener
- added J5: Conn_01x14_Socket, symbol Connector:Conn_01x14_Socket
Connections:
- net EXT_VREF: now also J5.5 (Pin_5)
- net GND: now also D2.2 (A), D3.2 (A), J5.14 (Pin_14)
- net IOB_0: now also J5.6 (Pin_6)
- net IOB_1: now also J5.7 (Pin_7)
- net IOB_2: now also J5.8 (Pin_8)
- net IOB_3: now also J5.9 (Pin_9)
- net IOB_4: now also J5.10 (Pin_10)
- net IOB_5: now also J5.11 (Pin_11)
- net IOB_6: now also J5.12 (Pin_12)
- net IOB_7: now also J5.13 (Pin_13)
- net VBUS: now also J5.3 (Pin_3), J5.4 (Pin_4)
- new net ADC0: D2.1 (K), J5.1 (Pin_1)
- new net ADC1: D3.1 (K), J5.2 (Pin_2)
Other:
- moved on the sheet: FB1

Commit message: update conn packages
Parts:
- added H1, H2, H3, H4, H5, H6: MountingHole, MountingHole:MountingHole_3.2mm_M3_Pad_TopOnly, symbol Mechanical:MountingHole
- D2, D3: footprint (none) -> Diode_SMD:D_0201_0603Metric
- J3, J4: footprint (none) -> Connector_Molex:Molex_PicoBlade_53261-0571_1x05-1MP_P1.25mm_Horizontal
- J5: footprint (none) -> Connector_FFC-FPC:Molex_200528-0130_1x13-1MP_P1.00mm_Horizontal
- R2, R3: footprint (none) -> Resistor_SMD:R_0603_1608Metric
Connections:
- no-connect marks 0 -> 1
Other:
- moved on the sheet: D2, D3
