File: hardware/goose60rev2/connector.kicad_sch (KiCad schematic)
At the start: 22 parts, among them J1 USB_C_Receptacle_USB2.0_14P, J3 Conn_01x04_Socket, J4 Conn_01x04_Socket, J5 Conn_01x14_Socket, U2 TXS0108EPW, U6 USBLC6-2SC6

Commit message: update goose60 rev2 PCB
Parts:
- removed D2, D3: 3.6V, Diode_SMD:D_0201_0603Metric, symbol Device:D_Zener
- removed J3: Conn_01x04_Socket, Connector_Molex:Molex_PicoBlade_53261-0571_1x05-1MP_P1.25mm_Horizontal, symbol Connector:Conn_01x04_Socket
- added D2, D3: BAT54S, Package_TO_SOT_SMD:SOT-23, symbol Diode:BAT54S
- added R12, R13: 0ohm, Resistor_SMD:R_0603_1608Metric, symbol Device:R
- added R16, R17: 10K, Resistor_SMD:R_0603_1608Metric, symbol Device:R_Small_US
- J4: renamed from J5; footprint Connector_FFC-FPC:Molex_200528-0130_1x13-1MP_P1.00mm_Horizontal -> Connector_FFC-FPC:Molex_200528-0140_1x14-1MP_P1.00mm_Horizontal
- renumbered J4 to J3
Connections:
- net ADC0: now also D2.3 (COM), R16.2; no longer J4.1 (Pin_1)
- net ADC1: now also D3.3 (COM), R17.2; no longer J4.2 (Pin_2)
- net EXT_VREF: now also J4.10 (Pin_10); no longer J4.5 (Pin_5)
- net GND: now also J4.1 (Pin_1), D2.1 (A), D3.1 (A); no longer J4.14 (Pin_14)
- net IOB_0: now also J4.2 (Pin_2); no longer J4.6 (Pin_6)
- net IOB_1: now also J4.3 (Pin_3); no longer J4.7 (Pin_7)
- net IOB_2: now also J4.4 (Pin_4); no longer J4.8 (Pin_8)
- net IOB_3: now also J4.5 (Pin_5); no longer J4.9 (Pin_9)
- net IOB_4: now also J4.6 (Pin_6); no longer J4.10 (Pin_10)
- net IOB_5: now also J4.7 (Pin_7); no longer J4.11 (Pin_11)
- net IOB_6: now also J4.8 (Pin_8); no longer J4.12 (Pin_12)
- net IOB_7: now also J4.9 (Pin_9); no longer J4.13 (Pin_13)
- net USBD+: now also J3.2 (Pin_2), R13.2; no longer J3.3 (Pin_3)
- net USBD-: now also J3.3 (Pin_3), R12.2; no longer J3.2 (Pin_2)
- net VBUS: now also J1.A4 (VBUS), J1.A9 (VBUS), J1.B4 (VBUS), J1.B9 (VBUS), J4.11 (Pin_11), J4.12 (Pin_12); no longer J4.3 (Pin_3), J4.4 (Pin_4)
- net VREF: now also D2.2 (K), D3.2 (K)
- net CON_D-: now reaches J1.A7 (D-), J1.B7 (D-)
- net CON_D-: now also R12.1
- net CON_D+: now reaches J1.A6 (D+), J1.B6 (D+)
- net CON_D+: now also R13.1
- new net ADC0_CON: J4.13 (Pin_13), R16.1
- new net ADC1_CON: J4.14 (Pin_14), R17.1
- no-connect marks 1 -> 0
Other:
- moved on the sheet: D61, J3, J4

Commit message: add stabilizer and remove 6u hhkb support
Parts:
- R12, R13: footprint Resistor_SMD:R_0603_1608Metric -> Resistor_SMD:R_0402_1005Metric
Changed lines of the file:
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@@
 			)
 		)
-		(property "Footprint" "Resistor_SMD:R_0603_1608Metric"
+		(property "Footprint" "Resistor_SMD:R_0402_1005Metric"
 			(at 91.44 60.198 90)
 			(effects
@@
 			)
 		)
-		(property "Footprint" "Resistor_SMD:R_0603_1608Metric"
+		(property "Footprint" "Resistor_SMD:R_0402_1005Metric"
 			(at 91.44 57.658 90)
 			(effects
