File: hardware/goose60rev2/goose60rev2.kicad_pcb (KiCad board)
At the start: 2 copper layers, 285 x 94.6 mm, 0 parts

Commit message: update goose60 rev2 PCB
Parts:
- added C1: 2.2u/6.3V, Capacitor_SMD:C_0603_1608Metric_Pad1.08x0.95mm_HandSolder, B.Cu at (162.8, 187.8)
- added C10: 1uF/16V, Capacitor_SMD:C_0603_1608Metric, B.Cu at (141.9, 139.5)
- added C11: 1uF/16V, Capacitor_SMD:C_0603_1608Metric, B.Cu at (150.8, 139.5)
- added C12: 100uF/16V, Capacitor_SMD:C_0603_1608Metric, B.Cu at (143.4, 139.5)
- added C13: 100u/6.3V, Capacitor_SMD:C_0603_1608Metric_Pad1.08x0.95mm_HandSolder, B.Cu at (167.3, 192.8)
- added C14: 100u/6.3V, Capacitor_SMD:C_0603_1608Metric_Pad1.08x0.95mm_HandSolder, B.Cu at (161.3, 190.9)
- added C15: 100n/6.3V, Capacitor_SMD:C_0603_1608Metric_Pad1.08x0.95mm_HandSolder, B.Cu at (161.3, 181.7)
- added C16: 15P/25V, Capacitor_SMD:C_0603_1608Metric_Pad1.08x0.95mm_HandSolder, B.Cu at (180.8, 182.3)
- added C17: 15P/25V, Capacitor_SMD:C_0603_1608Metric_Pad1.08x0.95mm_HandSolder, B.Cu at (183.8, 184.9)
- added C18: 2U2/6.3V, Capacitor_SMD:C_0603_1608Metric_Pad1.08x0.95mm_HandSolder, B.Cu at (159.7, 181.7)
- added C19: 100u/6.3V, Capacitor_SMD:C_0603_1608Metric_Pad1.08x0.95mm_HandSolder, B.Cu at (172.6, 178.2)
- added C2: 100n/6.3V, Capacitor_SMD:C_0603_1608Metric_Pad1.08x0.95mm_HandSolder, B.Cu at (162.8, 189.3)
- added C20: 47nF/16V, Capacitor_SMD:C_0603_1608Metric, B.Cu at (128.8, 160.7)
- added C21: 100u/6.3V, Capacitor_SMD:C_0603_1608Metric_Pad1.08x0.95mm_HandSolder, B.Cu at (162.3, 185.3)
- added C22: 0.1u/6.3V, Capacitor_SMD:C_0603_1608Metric_Pad1.08x0.95mm_HandSolder, B.Cu at (159.9, 138.9)
- added C3: 100u/6.3V, Capacitor_SMD:C_0603_1608Metric_Pad1.08x0.95mm_HandSolder, B.Cu at (167.9, 178.2)
- added C4: 2.2u/6.3V, Capacitor_SMD:C_0603_1608Metric_Pad1.08x0.95mm_HandSolder, B.Cu at (177.2, 192.8)
- added C5: 2.2u/6.3V, Capacitor_SMD:C_0603_1608Metric_Pad1.08x0.95mm_HandSolder, B.Cu at (161.3, 192.4)
- added C6: 100u/6.3V, Capacitor_SMD:C_0603_1608Metric_Pad1.08x0.95mm_HandSolder, B.Cu at (172.6, 192.8)
- added C7: 100u/6.3V, Capacitor_SMD:C_0603_1608Metric_Pad1.08x0.95mm_HandSolder, B.Cu at (180.9, 189.0)
- added C8: 100nF/16V, Capacitor_SMD:C_0603_1608Metric, B.Cu at (152.4, 139.5)
- added C9: 100nF/16V, Capacitor_SMD:C_0603_1608Metric, B.Cu at (144.9, 139.5)
- added D1: BAT54S, Package_TO_SOT_SMD:SOT-23, B.Cu at (134.8, 160.7)
- added D1_1: 1N4148, Diode_SMD:D_0805_2012Metric, B.Cu at (74.5, 106.0)
- added D1_10: 1N4148, Diode_SMD:D_0805_2012Metric, B.Cu at (245.0, 108.6)
- added D1_11: 1N4148, Diode_SMD:D_0805_2012Metric, B.Cu at (264.0, 108.6)
- added D1_12: 1N4148, Diode_SMD:D_0805_2012Metric, B.Cu at (283.1, 108.6)
- added D1_13: 1N4148, Diode_SMD:D_0805_2012Metric, B.Cu at (302.1, 108.6)
- added D1_2: 1N4148, Diode_SMD:D_0805_2012Metric, B.Cu at (92.6, 109.5)
- added D1_3: 1N4148, Diode_SMD:D_0805_2012Metric, B.Cu at (111.6, 108.6)
- added D1_4: 1N4148, Diode_SMD:D_0805_2012Metric, B.Cu at (130.7, 108.6)
- added D1_5: 1N4148, Diode_SMD:D_0805_2012Metric, B.Cu at (149.7, 108.6)
- added D1_6: 1N4148, Diode_SMD:D_0805_2012Metric, B.Cu at (168.8, 108.6)
- added D1_7: 1N4148, Diode_SMD:D_0805_2012Metric, B.Cu at (187.8, 108.6)
- added D1_8: 1N4148, Diode_SMD:D_0805_2012Metric, B.Cu at (206.9, 108.6)
- added D1_9: 1N4148, Diode_SMD:D_0805_2012Metric, B.Cu at (225.9, 108.6)
- added D2: BAT54S, Package_TO_SOT_SMD:SOT-23, B.Cu at (232.0, 192.4)
- added D2_1: 1N4148, Diode_SMD:D_0805_2012Metric, B.Cu at (79.3, 124.3)
- added D2_10: 1N4148, Diode_SMD:D_0805_2012Metric, B.Cu at (254.5, 126.6)
- added D2_11: 1N4148, Diode_SMD:D_0805_2012Metric, B.Cu at (273.6, 126.6)
- added D2_12: 1N4148, Diode_SMD:D_0805_2012Metric, B.Cu at (292.6, 126.6)
- added D2_13: 1N4148, Diode_SMD:D_0805_2012Metric, B.Cu at (311.6, 126.6)
- added D2_14: 1N4148, Diode_SMD:D_0805_2012Metric, B.Cu at (332.9, 118.3)
- added D2_2: 1N4148, Diode_SMD:D_0805_2012Metric, B.Cu at (102.1, 126.6)
- added D2_3: 1N4148, Diode_SMD:D_0805_2012Metric, B.Cu at (121.2, 126.6)
- added D2_4: 1N4148, Diode_SMD:D_0805_2012Metric, B.Cu at (140.2, 126.6)
- added D2_5: 1N4148, Diode_SMD:D_0805_2012Metric, B.Cu at (159.2, 126.6)
- added D2_6: 1N4148, Diode_SMD:D_0805_2012Metric, B.Cu at (178.3, 126.6)
- added D2_7: 1N4148, Diode_SMD:D_0805_2012Metric, B.Cu at (197.3, 126.6)
- added D2_8: 1N4148, Diode_SMD:D_0805_2012Metric, B.Cu at (216.4, 126.6)
- added D2_9: 1N4148, Diode_SMD:D_0805_2012Metric, B.Cu at (235.4, 126.6)
- added D3: BAT54S, Package_TO_SOT_SMD:SOT-23, B.Cu at (240.6, 192.4)
- added D3_1: 1N4148, Diode_SMD:D_0805_2012Metric, B.Cu at (81.9, 143.3)
- added D3_10: 1N4148, Diode_SMD:D_0805_2012Metric, B.Cu at (259.3, 145.5)
- added D3_11: 1N4148, Diode_SMD:D_0805_2012Metric, B.Cu at (278.4, 145.5)
- added D3_12: 1N4148, Diode_SMD:D_0805_2012Metric, B.Cu at (297.4, 145.5)
- added D3_13: 1N4148, Diode_SMD:D_0805_2012Metric, B.Cu at (324.3, 145.5)
- added D3_14: 1N4148, Diode_SMD:D_0805_2012Metric, B.Cu at (332.7, 137.8)
- added D3_2: 1N4148, Diode_SMD:D_0805_2012Metric, B.Cu at (106.9, 145.5)
- added D3_3: 1N4148, Diode_SMD:D_0805_2012Metric, B.Cu at (126.0, 145.5)
- added D3_4: 1N4148, Diode_SMD:D_0805_2012Metric, B.Cu at (140.9, 145.7)
- added D3_5: 1N4148, Diode_SMD:D_0805_2012Metric, B.Cu at (164.1, 145.5)
- added D3_6: 1N4148, Diode_SMD:D_0805_2012Metric, B.Cu at (183.1, 145.5)
- added D3_7: 1N4148, Diode_SMD:D_0805_2012Metric, B.Cu at (202.2, 145.5)
- added D3_8: 1N4148, Diode_SMD:D_0805_2012Metric, B.Cu at (221.2, 145.5)
- added D3_9: 1N4148, Diode_SMD:D_0805_2012Metric, B.Cu at (240.2, 145.5)
- added D4_1: 1N4148, Diode_SMD:D_0805_2012Metric, B.Cu at (86.6, 163.4)
- added D4_10: 1N4148, Diode_SMD:D_0805_2012Metric, B.Cu at (249.7, 165.3)
- added D4_11: 1N4148, Diode_SMD:D_0805_2012Metric, B.Cu at (268.8, 165.3)
- added D4_12: 1N4148, Diode_SMD:D_0805_2012Metric, B.Cu at (287.8, 165.3)
- added D4_13: 1N4148, Diode_SMD:D_0805_2012Metric, B.Cu at (307.6, 163.4)
- added D4_14: 1N4148, Diode_SMD:D_0805_2012Metric, B.Cu at (331.4, 171.7)
- added D4_3: 1N4148, Diode_SMD:D_0805_2012Metric, B.Cu at (116.4, 165.3)
- added D4_4: 1N4148, Diode_SMD:D_0805_2012Metric, B.Cu at (135.4, 165.3)
- added D4_5: 1N4148, Diode_SMD:D_0805_2012Metric, B.Cu at (150.2, 165.3)
- added D4_6: 1N4148, Diode_SMD:D_0805_2012Metric, B.Cu at (173.5, 165.3)
- added D4_7: 1N4148, Diode_SMD:D_0805_2012Metric, B.Cu at (192.6, 165.3)
- added D4_8: 1N4148, Diode_SMD:D_0805_2012Metric, B.Cu at (211.6, 165.3)
- added D4_9: 1N4148, Diode_SMD:D_0805_2012Metric, B.Cu at (230.7, 165.3)
- added D5_1: 1N4148, Diode_SMD:D_0805_2012Metric, B.Cu at (88.2, 192.7)
- added D5_11: 1N4148, Diode_SMD:D_0805_2012Metric, B.Cu at (259.8, 190.8)
- added D5_12: 1N4148, Diode_SMD:D_0805_2012Metric, B.Cu at (282.6, 191.7)
- added D5_13: 1N4148, Diode_SMD:D_0805_2012Metric, B.Cu at (306.3, 191.7)
- added D5_14: 1N4148, Diode_SMD:D_0805_2012Metric, B.Cu at (329.7, 191.7)
- added D5_2: 1N4148, Diode_SMD:D_0805_2012Metric, B.Cu at (93.6, 191.7)
- added D5_3: 1N4148, Diode_SMD:D_0805_2012Metric, B.Cu at (117.6, 191.7)
- added D5_7: 1N4148, Diode_SMD:D_0805_2012Metric, B.Cu at (219.8, 189.2)
- added D61: ESD5Zxx, Diode_SMD:D_SOD-523, B.Cu at (140.3, 139.4)
- added D62: 1N4148, Diode_SMD:D_SOD-323, B.Cu at (147.9, 142.2)
- added D_14: 1N4148, Diode_SMD:D_0805_2012Metric, B.Cu at (316.0, 108.6)
- added FB1: GZ2012D601TF, Inductor_SMD:L_0805_2012Metric, B.Cu at (76.0, 101.8)
- added H1: MountingHole, MountingHole:MountingHole_3.2mm_M3_Pad_TopOnly, F.Cu at (92.7, 128.2)
- added H2: MountingHole, MountingHole:MountingHole_3.2mm_M3_Pad_TopOnly, F.Cu at (195.7, 147.3)
- added H3: MountingHole, MountingHole:MountingHole_3.2mm_M3_Pad_TopOnly, F.Cu at (327.6, 128.2)
- added H4: MountingHole, MountingHole:MountingHole_3.2mm_M3_Pad_TopOnly, F.Cu at (69.0, 156.8)
- added H5: MountingHole, MountingHole:MountingHole_3.2mm_M3_Pad_TopOnly, F.Cu at (351.0, 156.8)
- added H6: MountingHole, MountingHole:MountingHole_3.2mm_M3_Pad_TopOnly, F.Cu at (258.0, 185.5)
- added J1: USB_C_Receptacle_USB2.0_14P, Connector_USB:USB_C_Receptacle_GCT_USB4105-xx-A_16P_TopMnt_Horizontal, B.Cu at (86.0, 101.8)
- added J2: Conn_01x04_Pin, Connector_PinHeader_2.54mm:PinHeader_1x04_P2.54mm_Vertical, F.Cu at (181.3, 179.1)
- added J3: Conn_01x04_Socket, Connector_Molex:Molex_PicoBlade_53261-0571_1x05-1MP_P1.25mm_Horizontal, B.Cu at (113.5, 139.6)
- added J4: Conn_01x14_Socket, Connector_FFC-FPC:Molex_200528-0140_1x14-1MP_P1.00mm_Horizontal, B.Cu at (235.1, 188.1)
- added R1: no-fit, Resistor_SMD:R_0603_1608Metric, B.Cu at (177.9, 184.9)
- added R10: 150K/1%, Resistor_SMD:R_0603_1608Metric, B.Cu at (130.4, 160.7)
- added R11: 1K, Resistor_SMD:R_0603_1608Metric, B.Cu at (95.0, 154.6)
- added R12: 0ohm, Resistor_SMD:R_0603_1608Metric, B.Cu at (108.2, 139.8)
- added R13: 0ohm, Resistor_SMD:R_0603_1608Metric, B.Cu at (108.2, 138.2)
- added R14: 1K, Resistor_SMD:R_0603_1608Metric, B.Cu at (180.8, 187.4)
- added R15: 22R/5%, Resistor_SMD:R_0603_1608Metric, B.Cu at (134.3, 157.8)
- added R16: 10K, Resistor_SMD:R_0603_1608Metric, B.Cu at (234.5, 192.5)
- added R17: 10K, Resistor_SMD:R_0603_1608Metric, B.Cu at (243.1, 192.5)
- added R18: 22R/5%, Resistor_SMD:R_0603_1608Metric, B.Cu at (134.3, 155.9)
- added R19: ~, Resistor_SMD:R_0603_1608Metric, B.Cu at (159.1, 141.3)
- added R2: 5.1K, Resistor_SMD:R_0603_1608Metric, B.Cu at (75.8, 103.5)
- added R24: 100R/5%, Resistor_SMD:R_0603_1608Metric, B.Cu at (146.9, 136.8)
- added R3: 5.1K, Resistor_SMD:R_0603_1608Metric, B.Cu at (94.5, 103.5)
- added R4: no-fit, Resistor_SMD:R_0603_1608Metric, B.Cu at (96.6, 154.6)
- added R5: 200R, Resistor_SMD:R_0603_1608Metric, B.Cu at (165.3, 190.1)
- added R6: 1R, Resistor_SMD:R_0603_1608Metric, B.Cu at (164.5, 192.4)
- added R7: no-fit, Resistor_SMD:R_0603_1608Metric, B.Cu at (219.4, 175.0)
- added R8: no-fit, Resistor_SMD:R_0603_1608Metric, B.Cu at (223.5, 175.0)
- added R9: 100K/1%, Resistor_SMD:R_0603_1608Metric, B.Cu at (132.0, 160.7)
- added REF**: Stabilizer_Cherry_MX_2.00u, Mounting_Keyboard_Stabilizer:Stabilizer_Cherry_MX_2.00u, F.Cu at (326.7, 166.7)
- added REF**: Stabilizer_Cherry_MX_2.00u, Mounting_Keyboard_Stabilizer:Stabilizer_Cherry_MX_2.00u, F.Cu at (333.8, 109.5)
- added REF**: Stabilizer_Cherry_MX_7.00u, Mounting_Keyboard_Stabilizer:Stabilizer_Cherry_MX_7.00u, F.Cu at (210.0, 185.7)
- added REF**: Stabilizer_Cherry_MX_2.00u, Mounting_Keyboard_Stabilizer:Stabilizer_Cherry_MX_2.00u, F.Cu at (331.4, 147.6)
- added REF**: Stabilizer_Cherry_MX_6.00u, Mounting_Keyboard_Stabilizer:Stabilizer_Cherry_MX_6.00u, F.Cu at (200.5, 185.7)
- added REF**: Stabilizer_Cherry_MX_2.00u, Mounting_Keyboard_Stabilizer:Stabilizer_Cherry_MX_2.00u, F.Cu at (88.6, 166.7)
- added REF**: Stabilizer_Cherry_MX_6.25u, Mounting_Keyboard_Stabilizer:Stabilizer_Cherry_MX_6.25u, F.Cu at (198.1, 185.7)
- added SW1: SW_Push, Button_Switch_SMD:SW_SPST_TL3342, B.Cu at (96.9, 148.5)
- added SW1_1: SW_Push, Switch_Keyboard_Hotswap_Kailh:SW_Hotswap_Kailh_MX_1.00u, F.Cu at (76.7, 109.5)
- added SW1_10: SW_Push, Switch_Keyboard_Hotswap_Kailh:SW_Hotswap_Kailh_MX_1.00u, F.Cu at (248.1, 109.5)
- added SW1_11: SW_Push, Switch_Keyboard_Hotswap_Kailh:SW_Hotswap_Kailh_MX_1.00u, F.Cu at (267.1, 109.5)
- added SW1_12: SW_Push, Switch_Keyboard_Hotswap_Kailh:SW_Hotswap_Kailh_MX_1.00u, F.Cu at (286.2, 109.5)
- added SW1_13: SW_Push, Switch_Keyboard_Hotswap_Kailh:SW_Hotswap_Kailh_MX_1.00u, F.Cu at (305.2, 109.5)
- added SW1_14: SW_Push, Switch_Keyboard_Hotswap_Kailh:SW_Hotswap_Kailh_MX_2.00u, F.Cu at (333.8, 109.5)
- added SW1_15: SW_Push, Switch_Keyboard_Hotswap_Kailh:SW_Hotswap_Kailh_MX_1.00u, F.Cu at (324.3, 109.5)
- added SW1_2: SW_Push, Switch_Keyboard_Hotswap_Kailh:SW_Hotswap_Kailh_MX_1.00u, F.Cu at (95.7, 109.5)
- added SW1_3: SW_Push, Switch_Keyboard_Hotswap_Kailh:SW_Hotswap_Kailh_MX_1.00u, F.Cu at (114.8, 109.5)
- added SW1_4: SW_Push, Switch_Keyboard_Hotswap_Kailh:SW_Hotswap_Kailh_MX_1.00u, F.Cu at (133.8, 109.5)
- added SW1_5: SW_Push, Switch_Keyboard_Hotswap_Kailh:SW_Hotswap_Kailh_MX_1.00u, F.Cu at (152.8, 109.5)
- added SW1_6: SW_Push, Switch_Keyboard_Hotswap_Kailh:SW_Hotswap_Kailh_MX_1.00u, F.Cu at (171.9, 109.5)
- added SW1_7: SW_Push, Switch_Keyboard_Hotswap_Kailh:SW_Hotswap_Kailh_MX_1.00u, F.Cu at (190.9, 109.5)
- added SW1_8: SW_Push, Switch_Keyboard_Hotswap_Kailh:SW_Hotswap_Kailh_MX_1.00u, F.Cu at (210.0, 109.5)
- added SW1_9: SW_Push, Switch_Keyboard_Hotswap_Kailh:SW_Hotswap_Kailh_MX_1.00u, F.Cu at (229.1, 109.5)
- added SW2_1: SW_Push, Switch_Keyboard_Hotswap_Kailh:SW_Hotswap_Kailh_MX_1.50u, F.Cu at (81.4, 128.6)
- added SW2_10: SW_Push, Switch_Keyboard_Hotswap_Kailh:SW_Hotswap_Kailh_MX_1.00u, F.Cu at (257.6, 128.6)
- added SW2_11: SW_Push, Switch_Keyboard_Hotswap_Kailh:SW_Hotswap_Kailh_MX_1.00u, F.Cu at (276.7, 128.6)
- added SW2_12: SW_Push, Switch_Keyboard_Hotswap_Kailh:SW_Hotswap_Kailh_MX_1.00u, F.Cu at (295.7, 128.6)
- added SW2_13: SW_Push, Switch_Keyboard_Hotswap_Kailh:SW_Hotswap_Kailh_MX_1.00u, F.Cu at (314.8, 128.6)
- added SW2_14: SW_Push, Switch_Keyboard_Hotswap_Kailh:SW_Hotswap_Kailh_MX_1.00u, F.Cu at (343.4, 109.5)
- added SW2_2: SW_Push, Switch_Keyboard_Hotswap_Kailh:SW_Hotswap_Kailh_MX_1.00u, F.Cu at (105.2, 128.6)
- added SW2_3: SW_Push, Switch_Keyboard_Hotswap_Kailh:SW_Hotswap_Kailh_MX_1.00u, F.Cu at (124.3, 128.6)
- added SW2_4: SW_Push, Switch_Keyboard_Hotswap_Kailh:SW_Hotswap_Kailh_MX_1.00u, F.Cu at (143.3, 128.6)
- added SW2_5: SW_Push, Switch_Keyboard_Hotswap_Kailh:SW_Hotswap_Kailh_MX_1.00u, F.Cu at (162.4, 128.6)
- added SW2_6: SW_Push, Switch_Keyboard_Hotswap_Kailh:SW_Hotswap_Kailh_MX_1.00u, F.Cu at (181.4, 128.6)
- added SW2_7: SW_Push, Switch_Keyboard_Hotswap_Kailh:SW_Hotswap_Kailh_MX_1.00u, F.Cu at (200.5, 128.6)
- added SW2_8: SW_Push, Switch_Keyboard_Hotswap_Kailh:SW_Hotswap_Kailh_MX_1.00u, F.Cu at (219.5, 128.6)
- added SW2_9: SW_Push, Switch_Keyboard_Hotswap_Kailh:SW_Hotswap_Kailh_MX_1.00u, F.Cu at (238.6, 128.6)
- added SW3_1: SW_Push, Switch_Keyboard_Hotswap_Kailh:SW_Hotswap_Kailh_MX_1.75u, F.Cu at (83.8, 147.6)
- added SW3_10: SW_Push, Switch_Keyboard_Hotswap_Kailh:SW_Hotswap_Kailh_MX_1.00u, F.Cu at (262.4, 147.6)
- added SW3_11: SW_Push, Switch_Keyboard_Hotswap_Kailh:SW_Hotswap_Kailh_MX_1.00u, F.Cu at (281.4, 147.6)
- added SW3_12: SW_Push, Switch_Keyboard_Hotswap_Kailh:SW_Hotswap_Kailh_MX_1.00u, F.Cu at (300.5, 147.6)
- added SW3_13: SW_Push, Switch_Keyboard_Hotswap_Kailh:SW_Hotswap_Kailh_MX_2.25u, F.Cu at (331.4, 147.6)
- added SW3_14: SW_Push, Switch_Keyboard_Hotswap_Kailh:SW_Hotswap_Kailh_MX_1.50u, F.Cu at (338.6, 128.6)
- added SW3_2: SW_Push, Switch_Keyboard_Hotswap_Kailh:SW_Hotswap_Kailh_MX_1.00u, F.Cu at (110.0, 147.6)
- added SW3_3: SW_Push, Switch_Keyboard_Hotswap_Kailh:SW_Hotswap_Kailh_MX_1.00u, F.Cu at (129.0, 147.6)
- added SW3_4: SW_Push, Switch_Keyboard_Hotswap_Kailh:SW_Hotswap_Kailh_MX_1.00u, F.Cu at (148.1, 147.6)
- added SW3_5: SW_Push, Switch_Keyboard_Hotswap_Kailh:SW_Hotswap_Kailh_MX_1.00u, F.Cu at (167.1, 147.6)
- added SW3_6: SW_Push, Switch_Keyboard_Hotswap_Kailh:SW_Hotswap_Kailh_MX_1.00u, F.Cu at (186.2, 147.6)
- added SW3_7: SW_Push, Switch_Keyboard_Hotswap_Kailh:SW_Hotswap_Kailh_MX_1.00u, F.Cu at (205.2, 147.6)
- added SW3_8: SW_Push, Switch_Keyboard_Hotswap_Kailh:SW_Hotswap_Kailh_MX_1.00u, F.Cu at (224.3, 147.6)
- added SW3_9: SW_Push, Switch_Keyboard_Hotswap_Kailh:SW_Hotswap_Kailh_MX_1.00u, F.Cu at (243.3, 147.6)
- added SW4_1: SW_Push, Switch_Keyboard_Hotswap_Kailh:SW_Hotswap_Kailh_MX_2.25u, F.Cu at (88.6, 166.7)
- added SW4_10: SW_Push, Switch_Keyboard_Hotswap_Kailh:SW_Hotswap_Kailh_MX_1.00u, F.Cu at (252.9, 166.7)
- added SW4_11: SW_Push, Switch_Keyboard_Hotswap_Kailh:SW_Hotswap_Kailh_MX_1.00u, F.Cu at (271.9, 166.7)
- added SW4_12: SW_Push, Switch_Keyboard_Hotswap_Kailh:SW_Hotswap_Kailh_MX_1.00u, F.Cu at (291.0, 166.7)
- added SW4_13: SW_Push, Switch_Keyboard_Hotswap_Kailh:SW_Hotswap_Kailh_MX_2.75u, F.Cu at (326.7, 166.7)
- added SW4_14: SW_Push, Switch_Keyboard_Hotswap_Kailh:SW_Hotswap_Kailh_MX_1.00u, F.Cu at (343.4, 166.7)
- added SW4_15: SW_Push, Switch_Keyboard_Hotswap_Kailh:SW_Hotswap_Kailh_MX_1.75u, F.Cu at (317.2, 166.7)
- added SW4_3: SW_Push, Switch_Keyboard_Hotswap_Kailh:SW_Hotswap_Kailh_MX_1.00u, F.Cu at (119.5, 166.7)
- added SW4_4: SW_Push, Switch_Keyboard_Hotswap_Kailh:SW_Hotswap_Kailh_MX_1.00u, F.Cu at (138.6, 166.7)
- added SW4_5: SW_Push, Switch_Keyboard_Hotswap_Kailh:SW_Hotswap_Kailh_MX_1.00u, F.Cu at (157.6, 166.7)
- added SW4_6: SW_Push, Switch_Keyboard_Hotswap_Kailh:SW_Hotswap_Kailh_MX_1.00u, F.Cu at (176.7, 166.7)
- added SW4_7: SW_Push, Switch_Keyboard_Hotswap_Kailh:SW_Hotswap_Kailh_MX_1.00u, F.Cu at (195.7, 166.7)
- added SW4_8: SW_Push, Switch_Keyboard_Hotswap_Kailh:SW_Hotswap_Kailh_MX_1.00u, F.Cu at (214.8, 166.7)
- added SW4_9: SW_Push, Switch_Keyboard_Hotswap_Kailh:SW_Hotswap_Kailh_MX_1.00u, F.Cu at (233.8, 166.7)
- added SW5_1: SW_Push, Switch_Keyboard_Hotswap_Kailh:SW_Hotswap_Kailh_MX_1.25u, F.Cu at (79.0, 185.7)
- added SW5_10: SW_Push, Switch_Keyboard_Hotswap_Kailh:SW_Hotswap_Kailh_MX_1.25u, F.Cu at (269.5, 185.7)
- added SW5_11: SW_Push, Switch_Keyboard_Hotswap_Kailh:SW_Hotswap_Kailh_MX_1.50u, F.Cu at (271.9, 185.7)
- added SW5_12: SW_Push, Switch_Keyboard_Hotswap_Kailh:SW_Hotswap_Kailh_MX_1.25u, F.Cu at (293.3, 185.7)
- added SW5_13: SW_Push, Switch_Keyboard_Hotswap_Kailh:SW_Hotswap_Kailh_MX_1.50u, F.Cu at (291.0, 185.7)
- added SW5_14: SW_Push, Switch_Keyboard_Hotswap_Kailh:SW_Hotswap_Kailh_MX_1.00u, F.Cu at (295.7, 185.7)
- added SW5_15: SW_Push, Switch_Keyboard_Hotswap_Kailh:SW_Hotswap_Kailh_MX_1.25u, F.Cu at (317.2, 185.7)
- added SW5_16: SW_Push, Switch_Keyboard_Hotswap_Kailh:SW_Hotswap_Kailh_MX_1.00u, F.Cu at (314.8, 185.7)
- added SW5_17: SW_Push, Switch_Keyboard_Hotswap_Kailh:SW_Hotswap_Kailh_MX_1.25u, F.Cu at (341.0, 185.7)
- added SW5_18: SW_Push, Switch_Keyboard_Hotswap_Kailh:SW_Hotswap_Kailh_MX_1.50u, F.Cu at (338.6, 185.7)
- added SW5_2: SW_Push, Switch_Keyboard_Hotswap_Kailh:SW_Hotswap_Kailh_MX_1.25u, F.Cu at (102.8, 185.7)
- added SW5_3: SW_Push, Switch_Keyboard_Hotswap_Kailh:SW_Hotswap_Kailh_MX_1.25u, F.Cu at (126.7, 185.7)
- added SW5_4: SW_Push, Switch_Keyboard_Hotswap_Kailh:SW_Hotswap_Kailh_MX_1.50u, F.Cu at (81.4, 185.7)
- added SW5_5: SW_Push, Switch_Keyboard_Hotswap_Kailh:SW_Hotswap_Kailh_MX_1.00u, F.Cu at (105.2, 185.7)
- added SW5_6: SW_Push, Switch_Keyboard_Hotswap_Kailh:SW_Hotswap_Kailh_MX_1.50u, F.Cu at (129.0, 185.7)
- added SW5_7: SW_Push, Switch_Keyboard_Hotswap_Kailh:SW_Hotswap_Kailh_MX_6.25u, F.Cu at (198.1, 185.7)
- added SW5_8: SW_Push, Switch_Keyboard_Hotswap_Kailh:SW_Hotswap_Kailh_MX_7.00u, F.Cu at (210.0, 185.7)
- added SW5_9: SW_Push, Switch_Keyboard_Hotswap_Kailh:SW_Hotswap_Kailh_MX_6.00u, F.Cu at (200.5, 185.7)
- added TH1: Thermistor_NTC, Resistor_SMD:R_0603_1608Metric, B.Cu at (158.2, 138.9)
- added U1: RP2040, Package_DFN_QFN:QFN-56-1EP_7x7mm_P0.4mm_EP3.2x3.2mm, B.Cu at (171.1, 185.3)
- added U2: TXS0108EPW, Package_SO:TSSOP-20_4.4x6.5mm_P0.65mm, B.Cu at (221.4, 179.5)
- added U3: W25Q16JVSS, Package_SON:Winbond_USON-8-1EP_3x2mm_P0.5mm_EP0.2x1.6mm, B.Cu at (163.4, 181.1)
- added U6: USBLC6-2SC6, Package_TO_SOT_SMD:SOT-23-6, B.Cu at (130.4, 156.8)
- added U7: TLV75533PDBV, Package_TO_SOT_SMD:SOT-23-5, B.Cu at (147.9, 139.3)
- added X1: 12MHz, Crystal:Crystal_SMD_TXC_7M-4Pin_3.2x2.5mm, B.Cu at (180.8, 184.9)
Routing:
- net GND: track 0.00 -> 525.9 mm, vias 0 -> 28
- net row3: track 0.00 -> 376.8 mm, vias 0 -> 17
- net +3.3V: track 0.00 -> 368.9 mm, vias 0 -> 19
- net row1: track 0.00 -> 343.1 mm, vias 0 -> 15
- net row4: track 0.00 -> 342.8 mm, vias 0 -> 16
- net row2: track 0.00 -> 334.6 mm, vias 0 -> 15
- net col14: track 0.00 -> 293.9 mm, vias 0 -> 2
- net VIN: track 0.00 -> 287.6 mm, vias 0 -> 10
- net row5: track 0.00 -> 262.8 mm, vias 0 -> 8
- net col13: track 0.00 -> 257.7 mm, vias 0 -> 2
- net col12: track 0.00 -> 229.7 mm, vias 0 -> 2
- net col11: track 0.00 -> 200.2 mm, vias 0 -> 2
- net col1: track 0.00 -> 175.2 mm, vias 0 -> 2
- net col2: track 0.00 -> 162.9 mm, vias 0 -> 4
- net col10: track 0.00 -> 159.8 mm, vias 0 -> 2
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Other:
- board size 285 x 94.6 mm -> 285 x 95.1 mm
- board text added: "注意事項 3. Level shift 可能需要更換封裝 5. reset key 的封裝需要更改 6. Program Flash 的位置需要調整，最好是重新設計布局，盡可能讓 QSPI 等常，並整合 3.3V 線路，來縮減空間。 7. USB_VDD 電壓需要確認是否可以正常運作，目前是用 3.3V，但直覺是要用 5V"

Commit message: [WIP] update PCB layout
Routing:
- added copper zone on B.Cu, net GND
- added copper zone on F.Cu, net GND
Other:
- board text added: "2026.08.04"
- board text added: "Goose60 rev2"
- board text added: "rev2"
- board text removed: "注意事項 3. Level shift 可能需要更換封裝 5. reset key 的封裝需要更改 6. Program Flash 的位置需要調整，最好是重新設計布局，盡可能讓 QSPI 等常，並整合 3.3V 線路，來縮減空間。 7. USB_VDD 電壓需要確認是否可以正常運作，目前是用 3.3V，但直覺是要用 5V"
Changed lines of the file:
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@@
 		(layer "Edge.Cuts")
 	)
-	(gr_text "注意事項\n3. Level shift 可能需要更換封裝\n5. reset key 的封裝需要更改\n6. Program Flash 的位置需要調整，最好是重新設計布局，盡可能讓 QSPI 等常，並整合 3.3V 線路，來縮減空間。\n7. USB_VDD 電壓需要確認是否可以正常運作，目前是用 3.3V，但直覺是要用 5V\n"
-		(at 108.8 230.11 0)
+	(gr_text "2026.08.04"
+		(at 332.26 281.08 0)
+		(layer "Cmts.User")
+		(effects
+			(font
+				(size 1.5 1.5)
+				(thickness 0.2)
+			)
+			(justify left bottom)
+		)
+	)
+	(gr_text "rev2"
+		(at 392.69 280.96 0)
+		(layer "Cmts.User")
+		(effects
+			(font
+				(size 1.5 1.5)
+				(thickness 0.2)
+			)
+			(justify left bottom)
+		)
+	)
+	(gr_text "Goose60 rev2"
+		(at 317.69 277.66 0)
 		(layer "Cmts.User")
 		(effects
 			(font
 				(size 2 2)
-				(thickness 0.15)
+				(thickness 0.3)
 			)
 			(justify left bottom)
 		)
 	)
-	(gr_text_box "PCB中心點\nX: 210\nY: 147.6\n\n衛星軸孔已經定位。\n確定支援下列布局\n- default 60%\n- WK 60%\n- WKL 60%\n- HHKB 6u\n- HHKB 7u\n\nPCB 製程能力參考 https://www.pcb.ing/ability"
+	(gr_text "Goose60 rev2"
+		(at 314.27 266.39 0)
+		(layer "Cmts.User")
+		(effects
+			(font
+				(size 8 8)
+				(thickness 1)
+			)
+			(justify left bottom)
+		)
+	)
+	(gr_text_box "PCB中心點\nX: 210\nY: 147.6\n\n衛星軸孔已經定位。\n確定支援下列布局\n- default 60%\n- WK 60%\n- WKL 60%\n- HHKB 6u\n- HHKB 7u"
 		(start 280.685 19.71)
-		(end 397.115 90.75)
+		(end 397.115 78.73)
 		(margins 1.0025 1.0025 1.0025 1.0025)
 		(layer "Cmts.User")
@@
 		(net 136)
 	)
+	(zone
+		(net 1)
+		(net_name "GND")
+		(layers "F.Cu" "B.Cu")
+		(hatch edge 0.5)
+		(connect_pads
+			(clearance 0.5)
+		)
+		(min_thickness 0.25)
+		(filled_areas_thickness no)
+		(fill yes
+			(thermal_gap 0.5)
+			(thermal_bridge_width 0.5)
+			(smoothing fillet)
+		)
+		(polygon
+			(pts
+				(xy 63.42 98.05) (xy 61.83 200.63) (xy 360.07 197.9) (xy 359.62 94.86) (xy 64.28 98.03)
+			)
+		)
+	)
 	(generated

Commit message: update rev2 PCB layout
Parts:
- removed the REF** at (331.4, 147.6)
Routing:
- net GNDPWR: track 13.4 -> 22.0 mm
- net col7: track 155.4 -> 154.8 mm
- net GND: vias 28 -> 679
Other:
- board text added: "2026.08.22"
- board text added: "JYKB"
- board text added: "Made in Taiwan."
- board text removed: "2026.08.04"

Commit message: update goose60 rev2 schematic and PCB layout
Parts:
- removed R1: no-fit, Resistor_SMD:R_0603_1608Metric
- added R20: 10K, Resistor_SMD:R_0603_1608Metric, B.Cu at (181.8, 193.1)
- added R21: 10K ~ 100K, Resistor_SMD:R_0603_1608Metric, B.Cu at (183.5, 190.5)
- moved C16 1.00 mm to (181.8, 182.3)
- moved C17 1.00 mm to (184.8, 184.9)
- moved R14 1.00 mm to (181.8, 187.4)
- moved X1 1.00 mm to (181.8, 184.9)
- moved C7 0.74 mm to (181.0, 189.8)
Connections:
- J2 pad 2: SWCLK -> GND
- J2 pad 3: GND -> SWCLK
Routing:
- net GND: track 525.9 -> 550.2 mm, vias 679 -> 721
- net +3.3V: track 368.9 -> 375.1 mm
- net SWCLK: track 26.0 -> 28.2 mm
- net SWDIO: track 26.6 -> 28.9 mm
- net XOUT: track 6.52 -> 7.52 mm
- net XIN: track 7.36 -> 8.36 mm
