File: hardware/goose60rev2/goose60rev2.kicad_pcb (KiCad board)
At the start: 2 copper layers, 285 x 95.1 mm, 211 parts, among them J1 USB_C_Receptacle_USB2.0_14P, J2 Conn_01x04_Pin, J3 Conn_01x04_Socket, J4 Conn_01x14_Socket, SW1 SW_Push, SW1_1 SW_Push, SW1_10 SW_Push, SW1_11 SW_Push, SW1_12 SW_Push, SW1_13 SW_Push, SW1_14 SW_Push, SW1_15 SW_Push, SW1_2 SW_Push, SW1_3 SW_Push, SW1_4 SW_Push, SW1_5 SW_Push, SW1_6 SW_Push, SW1_7 SW_Push, SW1_8 SW_Push, SW1_9 SW_Push, SW2_1 SW_Push, SW2_10 SW_Push, SW2_11 SW_Push, SW2_12 SW_Push, SW2_13 SW_Push, SW2_14 SW_Push, SW2_2 SW_Push, SW2_3 SW_Push, SW2_4 SW_Push, SW2_5 SW_Push, SW2_6 SW_Push, SW2_7 SW_Push, SW2_8 SW_Push, SW2_9 SW_Push, SW3_1 SW_Push, SW3_10 SW_Push, SW3_11 SW_Push, SW3_12 SW_Push, SW3_13 SW_Push, SW3_14 SW_Push, SW3_2 SW_Push, SW3_3 SW_Push, SW3_4 SW_Push, SW3_5 SW_Push, SW3_6 SW_Push, SW3_7 SW_Push, SW3_8 SW_Push, SW3_9 SW_Push, SW4_1 SW_Push, SW4_10 SW_Push, SW4_11 SW_Push, SW4_12 SW_Push, SW4_13 SW_Push, SW4_14 SW_Push, SW4_15 SW_Push, SW4_3 SW_Push, SW4_4 SW_Push, SW4_5 SW_Push, SW4_6 SW_Push, SW4_7 SW_Push, SW4_8 SW_Push, SW4_9 SW_Push, SW5_1 SW_Push, SW5_10 SW_Push, SW5_11 SW_Push, SW5_12 SW_Push, SW5_13 SW_Push, SW5_14 SW_Push, SW5_15 SW_Push, SW5_16 SW_Push, SW5_17 SW_Push, SW5_18 SW_Push, SW5_2 SW_Push, SW5_3 SW_Push, SW5_4 SW_Push, SW5_5 SW_Push, SW5_6 SW_Push, SW5_7 SW_Push, SW5_8 SW_Push, SW5_9 SW_Push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

Commit message: update PCB and export BOM
Parts:
- removed REF** (x3): Stabilizer_Cherry_MX_2.00u, Mounting_Keyboard_Stabilizer:Stabilizer_Cherry_MX_2.00u
- removed REF**: Stabilizer_Cherry_MX_7.00u, Mounting_Keyboard_Stabilizer:Stabilizer_Cherry_MX_7.00u
- removed REF**: Stabilizer_Cherry_MX_6.00u, Mounting_Keyboard_Stabilizer:Stabilizer_Cherry_MX_6.00u
- removed REF**: Stabilizer_Cherry_MX_6.25u, Mounting_Keyboard_Stabilizer:Stabilizer_Cherry_MX_6.25u
Routing:
- net GND: vias 740 -> 741

Commit message: add stabilizer and remove 6u hhkb support
Parts:
- removed SW5_14: SW_Push, Switch_Keyboard_Hotswap_Kailh:SW_Hotswap_Kailh_MX_1.00u
- removed SW5_9: SW_Push, Switch_Keyboard_Hotswap_Kailh:SW_Hotswap_Kailh_MX_6.00u
- added REF**: Stabilizer_Cherry_MX_2.00u, Mounting_Keyboard_Stabilizer:Stabilizer_Cherry_MX_2.00u, F.Cu at (331.4, 147.6)
- added REF**: Stabilizer_Cherry_MX_2.00u, Mounting_Keyboard_Stabilizer:Stabilizer_Cherry_MX_2.00u, F.Cu at (88.6, 166.7)
- added REF**: Stabilizer_Cherry_MX_7.00u, Mounting_Keyboard_Stabilizer:Stabilizer_Cherry_MX_7.00u, F.Cu at (210.0, 185.7)
- added REF**: Stabilizer_Cherry_MX_2.00u, Mounting_Keyboard_Stabilizer:Stabilizer_Cherry_MX_2.00u, F.Cu at (326.7, 166.7)
- added REF**: Stabilizer_Cherry_MX_6.25u, Mounting_Keyboard_Stabilizer:Stabilizer_Cherry_MX_6.25u, F.Cu at (198.1, 185.7)
- added REF**: Stabilizer_Cherry_MX_2.00u, Mounting_Keyboard_Stabilizer:Stabilizer_Cherry_MX_2.00u, F.Cu at (333.8, 109.5)
- R12, R13: footprint Resistor_SMD:R_0603_1608Metric -> Resistor_SMD:R_0402_1005Metric
- moved R13 1.86 mm to (110.0, 138.4)
- moved R12 1.85 mm to (110.0, 139.6)
Routing:
- net col12: track 229.7 -> 219.0 mm
- net Net-(D5_12-A): track 21.2 -> 13.1 mm
- net USBD-: track 36.4 -> 34.2 mm
- net /connector/CON_D+: track 49.4 -> 51.5 mm
- net /connector/CON_D-: track 50.1 -> 52.1 mm
- net Net-(D5_7-A): track 41.2 -> 39.3 mm
- net USBD+: track 36.3 -> 34.6 mm
- net QSPI_SS: track 95.4 -> 94.5 mm
- net GND: vias 741 -> 770
