File: hardware/goose60rev2/goose60rev2.kicad_sch (KiCad schematic)
At the start: 19 parts, among them J2 Conn_01x04_Pin, U1 RP2040, X1 12MHz

Commit message: update goose60 rev2 PCB
Parts:
- added C21: 100u/6.3V, Capacitor_SMD:C_0603_1608Metric_Pad1.08x0.95mm_HandSolder, symbol Device:C
- added C22: 0.1u/6.3V, Capacitor_SMD:C_0603_1608Metric_Pad1.08x0.95mm_HandSolder, symbol Device:C
- added R19: ~, Resistor_SMD:R_0603_1608Metric, symbol Device:R
- added TH1: Thermistor_NTC, Resistor_SMD:R_0603_1608Metric, symbol Device:Thermistor_NTC
Connections:
- net SPI0_CSn/UART0_RX/I2C0_SCL is gone; now on net col5: U1.3 (GPIO1)
- net SPI0_CSn/UART1_RX/I2C0_SCL is gone; now on net col7: U1.7 (GPIO5)
- net SPI0_RX/UART0_TX/I2C0_SDA is gone; now on net col4: U1.2 (GPIO0)
- net SPI0_RX/UART1_TX/I2C0_SDA is gone; now on net col6: U1.6 (GPIO4)
- net SPI0_SCK/UART0_CTS/I2C1_SDA is gone; now on net row1: U1.4 (GPIO2)
- net SPI0_TX/UART0_RTS/I2C1_SCL is gone; now on net row2: U1.5 (GPIO3)
- net +3V3: now also C21.1, R19.1
- net GND: now also C21.2, C22.1, TH1.2
- net SUBPWR_EN: now also U1.17 (GPIO14); no longer U1.37 (GPIO25)
- net VIN_ADC: no longer U1.39 (GPIO27_ADC1)
- net col1: now also U1.35 (GPIO23); no longer U1.8 (GPIO6)
- net col2: now also U1.34 (GPIO22); no longer U1.9 (GPIO7)
- net col3: now also U1.32 (GPIO21); no longer U1.11 (GPIO8)
- net col4: no longer U1.12 (GPIO9)
- net col5: no longer U1.13 (GPIO10)
- net col6: no longer U1.14 (GPIO11)
- net col7: no longer U1.15 (GPIO12)
- net col8: now also U1.8 (GPIO6); no longer U1.16 (GPIO13)
- net col9: now also U1.9 (GPIO7); no longer U1.17 (GPIO14)
- net row1: no longer U1.31 (GPIO20)
- net row2: no longer U1.32 (GPIO21)
- net row3: now also U1.36 (GPIO24); no longer U1.34 (GPIO22)
- net row4: now also U1.37 (GPIO25); no longer U1.35 (GPIO23)
- net row5: now also U1.31 (GPIO20); no longer U1.36 (GPIO24)
- net GPIO29_ADC3 renamed PCBA_NTC
- net PCBA_NTC: now also C22.2, R19.2, TH1.1
- new net GPIO29_ADC1: U1.39 (GPIO27_ADC1)
- new net SPI1_CSn/UART0_RX/I2C0_SCL: U1.16 (GPIO13)
- new net SPI1_CSn/UART1_RX/I2C0_SCL: U1.12 (GPIO9)
- new net SPI1_RX/UART0_TX/I2C0_SDA: U1.15 (GPIO12)
- new net SPI1_RX/UART1_TX/I2C0_SDA: U1.11 (GPIO8)
- new net SPI1_SCK/UART1_CTS/I2C1_SDA: U1.13 (GPIO10)
- new net SPI1_TX/UART1_RTS/I2C1_SCL: U1.14 (GPIO11)
Other:
- moved on the sheet: C13, C14, C19, C3, C6, C7, J2

Commit message: [WIP] update PCB layout
Other:
- note added: "2025.11.12"
- note added: "Goose60 rev2"
- note added: "rev2"
Changed lines of the file:
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@@
+		)
+	)
+	(text "2025.11.12"
+		(exclude_from_sim no)
+		(at 212.852 193.294 0)
+		(effects
+			(font
+				(size 1.27 1.27)
+				(thickness 0.508)
+				(bold yes)
+			)
+		)
+	)
+	(text "Goose60 rev2"
+		(exclude_from_sim no)
+		(at 199.136 174.244 0)
+		(effects
+			(font
+				(size 2.54 2.54)
+				(thickness 0.508)
+				(bold yes)
+			)
+		)
+	)
+	(text "rev2"
+		(exclude_from_sim no)
+		(at 272.796 193.294 0)
+		(effects
+			(font
+				(size 1.27 1.27)
+				(thickness 0.508)
+				(bold yes)
+			)
+		)
+	)
+	(text "Goose60 rev2"
+		(exclude_from_sim no)
+		(at 197.104 189.738 0)
+		(effects
+			(font
+				(size 1.778 1.778)
+				(thickness 0.508)
+				(bold yes)
+			)
 		)
 	)

Commit message: update goose60 rev2 schematic and PCB layout
Parts:
- removed R1: no-fit, Resistor_SMD:R_0603_1608Metric, symbol Device:R
- added R20: 10K, Resistor_SMD:R_0603_1608Metric, symbol Device:R
- added R21: 10K ~ 100K, Resistor_SMD:R_0603_1608Metric, symbol Device:R
Connections:
- net +3V3: now also R20.1
- net GND: now also J2.2 (Pin_2), R21.2; no longer J2.3 (Pin_3)
- net SWCLK: now also J2.3 (Pin_3), R21.1; no longer J2.2 (Pin_2)
- net SWDIO: now also R20.2
Other:
- moved on the sheet: J2
