File: hardware/goose60rev2/key_matrix.kicad_sch (KiCad schematic)
At the start: 139 parts, among them SW1_1 SW_Push, SW1_10 SW_Push, SW1_11 SW_Push, SW1_12 SW_Push, SW1_13 SW_Push, SW1_14 SW_Push, SW1_15 SW_Push, SW1_2 SW_Push, SW1_3 SW_Push, SW1_4 SW_Push, SW1_5 SW_Push, SW1_6 SW_Push, SW1_7 SW_Push, SW1_8 SW_Push, SW1_9 SW_Push, SW2_1 SW_Push, SW2_10 SW_Push, SW2_11 SW_Push, SW2_12 SW_Push, SW2_13 SW_Push, SW2_14 SW_Push, SW2_15 SW_Push, SW2_2 SW_Push, SW2_3 SW_Push, SW2_4 SW_Push, SW2_5 SW_Push, SW2_6 SW_Push, SW2_7 SW_Push, SW2_8 SW_Push, SW2_9 SW_Push, SW3_1 SW_Push, SW3_10 SW_Push, SW3_11 SW_Push, SW3_12 SW_Push, SW3_13 SW_Push, SW3_14 SW_Push, SW3_2 SW_Push, SW3_3 SW_Push, SW3_4 SW_Push, SW3_5 SW_Push, SW3_6 SW_Push, SW3_7 SW_Push, SW3_8 SW_Push, SW3_9 SW_Push, SW4_1 SW_Push, SW4_10 SW_Push, SW4_11 SW_Push, SW4_12 SW_Push, SW4_13 SW_Push, SW4_14 SW_Push, SW4_15 SW_Push, SW4_3 SW_Push, SW4_4 SW_Push, SW4_5 SW_Push, SW4_6 SW_Push, SW4_7 SW_Push, SW4_8 SW_Push, SW4_9 SW_Push, SW5_1 SW_Push, SW5_10 SW_Push, SW5_11 SW_Push, SW5_12 SW_Push, SW5_13 SW_Push, SW5_14 SW_Push, SW5_15 SW_Push, SW5_16 SW_Push, SW5_17 SW_Push, SW5_18 SW_Push, SW5_2 SW_Push, SW5_3 SW_Push, SW5_4 SW_Push, SW5_5 SW_Push, SW5_6 SW_Push, SW5_7 SW_Push, SW5_8 SW_Push, SW5_9 SW_Push

Commit message: update goose60 rev2 PCB
Parts:
- removed SW2_15: SW_Push, Switch_Keyboard_Hotswap_Kailh:SW_Hotswap_Kailh_MX_1.50u, symbol Switch:SW_Push
- SW1_15: footprint Switch_Keyboard_Hotswap_Kailh:SW_Hotswap_Kailh_MX_2.00u -> Switch_Keyboard_Hotswap_Kailh:SW_Hotswap_Kailh_MX_1.00u
- SW2_14: footprint Switch_Keyboard_Hotswap_Kailh:SW_Hotswap_Kailh_MX_1.50u -> Switch_Keyboard_Hotswap_Kailh:SW_Hotswap_Kailh_MX_1.00u
- SW3_14: footprint Switch_Keyboard_Hotswap_Kailh:SW_Hotswap_Kailh_MX_2.25u -> Switch_Keyboard_Hotswap_Kailh:SW_Hotswap_Kailh_MX_1.50u
- SW4_14: footprint Switch_Keyboard_Hotswap_Kailh:SW_Hotswap_Kailh_MX_2.75u -> Switch_Keyboard_Hotswap_Kailh:SW_Hotswap_Kailh_MX_1.00u
- SW4_15: footprint Switch_Keyboard_Hotswap_Kailh:SW_Hotswap_Kailh_MX_2.75u -> Switch_Keyboard_Hotswap_Kailh:SW_Hotswap_Kailh_MX_1.75u
- SW5_11, SW5_13, SW5_18, SW5_4, SW5_6: footprint Switch_Keyboard_Hotswap_Kailh:SW_Hotswap_Kailh_MX_1.25u -> Switch_Keyboard_Hotswap_Kailh:SW_Hotswap_Kailh_MX_1.50u
- SW5_14, SW5_16, SW5_5: footprint Switch_Keyboard_Hotswap_Kailh:SW_Hotswap_Kailh_MX_1.25u -> Switch_Keyboard_Hotswap_Kailh:SW_Hotswap_Kailh_MX_1.00u
- SW5_8: footprint Switch_Keyboard_Hotswap_Kailh:SW_Hotswap_Kailh_MX_6.25u -> Switch_Keyboard_Hotswap_Kailh:SW_Hotswap_Kailh_MX_7.00u
- SW5_9: footprint Switch_Keyboard_Hotswap_Kailh:SW_Hotswap_Kailh_MX_6.25u -> Switch_Keyboard_Hotswap_Kailh:SW_Hotswap_Kailh_MX_6.00u
Connections:
- net col1: now also SW5_4.2; no longer SW5_4.1
- net col11: now also SW5_11.2; no longer SW5_11.1
- net col12: now also SW5_13.2; no longer SW5_13.1
- net col13: now also SW4_13.2, SW5_16.2; no longer SW4_13.1, SW5_16.1
- net col14: now also SW1_14.2, SW5_18.2; no longer SW1_14.1, SW5_18.1
- net col2: now also SW5_5.2; no longer SW5_5.1
- net col3: now also SW5_6.2; no longer SW5_6.1
- net col7: now also SW5_8.2, SW5_9.2; no longer SW5_8.1, SW5_9.1
- net at D5_1.2 (A), SW5_1.2: now also SW5_4.1; no longer SW5_4.2
- net at D5_3.2 (A), SW5_3.2: now also SW5_6.1; no longer SW5_6.2
- net at D5_12.2 (A), SW5_12.2, SW5_14.2: now also SW5_13.1; no longer SW5_13.2
- net at D4_13.2 (A), SW4_15.2: now also SW4_13.1; no longer SW4_13.2
- net at D5_2.2 (A), SW5_2.2: now also SW5_5.1; no longer SW5_5.2
- net at D5_7.2 (A), SW5_7.2: now also SW5_8.1, SW5_9.1; no longer SW5_8.2, SW5_9.2
- net at D_14.2 (A), SW1_15.2: now also SW1_14.1; no longer SW1_14.2
- net at D5_13.2 (A), SW5_15.2: now also SW5_16.1; no longer SW5_16.2
- net at D5_11.2 (A), SW5_10.2: now also SW5_11.1; no longer SW5_11.2
- net at D5_14.2 (A), SW5_17.2: now also SW5_18.1; no longer SW5_18.2
Other:
- note added: "\ BS [HHKB]"
- note added: "` ~ [HHKB]"
- note removed: "BS [HHKB]"
- note removed: "\ ` ~ [HHKB]"
- moved on the sheet: SW1_14, SW4_13, SW5_11, SW5_13, SW5_16, SW5_18, SW5_4, SW5_5, SW5_6, SW5_8, SW5_9
Changed lines of the file:
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@@
 		)
 	)
-	(text "\\\n` ~ [HHKB]"
+	(text "` ~ [HHKB]"
 		(exclude_from_sim no)
 		(at 377.952 124.968 0)
@@
 		)
 	)
-	(text "BS [HHKB]"
+	(text "\\\nBS [HHKB]"
 		(exclude_from_sim no)
 		(at 387.35 161.29 0)
@@
 	)
 	(junction
-		(at 388.62 111.76)
-		(diameter 0)
-		(color 0 0 0 0)
-	)
-	(junction
 		(at 132.08 53.34)
 		(diameter 0)
@@
 	)
 	(junction
-		(at 367.03 104.14)
-		(diameter 0)
-		(color 0 0 0 0)
-	)
-	(junction
 		(at 161.29 184.15)
 		(diameter 0)
@@
 	(wire
 		(pts
-			(xy 367.03 104.14) (xy 367.03 111.76)
-		)
-		(stroke
-			(width 0)
-			(type default)
-		)
-	)
-	(wire
-		(pts
 			(xy 351.79 135.89) (xy 344.17 135.89)
 		)
@@
 	(wire
 		(pts
-			(xy 369.57 111.76) (xy 367.03 111.76)
-		)
-		(stroke
-			(width 0)
-			(type default)
-		)
-	)
-	(wire
-		(pts
 			(xy 311.15 184.15) (xy 313.69 184.15)
 		)
@@
 	(wire
 		(pts
-			(xy 388.62 111.76) (xy 388.62 114.3)
-		)
-		(stroke
-			(width 0)
-			(type default)
-		)
-	)
-	(wire
-		(pts
 			(xy 45.72 59.69) (xy 45.72 69.85)
 		)
@@
 	(wire
 		(pts
-			(xy 388.62 111.76) (xy 388.62 104.14)
+			(xy 388.62 104.14) (xy 388.62 114.3)
 		)
 		(stroke
@@
 	(wire
 		(pts
-			(xy 379.73 111.76) (xy 388.62 111.76)
-		)
-		(stroke
-			(width 0)
-			(type default)
-		)
-	)
-	(wire
-		(pts
 			(xy 274.32 184.15) (xy 275.59 184.15)
 		)
@@
 			)
 		)
-		(property "Footprint" "Switch_Keyboard_Hotswap_Kailh:SW_Hotswap_Kailh_MX_1.50u"
+		(property "Footprint" "Switch_Keyboard_Hotswap_Kailh:SW_Hotswap_Kailh_MX_1.00u"
 			(at 378.46 109.22 0)
 			(effects
@@
 			)
 		)
-		(property "Footprint" "Switch_Keyboard_Hotswap_Kailh:SW_Hotswap_Kailh_MX_1.25u"
+		(property "Footprint" "Switch_Keyboard_Hotswap_Kailh:SW_Hotswap_Kailh_MX_1.00u"
 			(at 325.12 234.95 0)
 			(effects
@@
 			)
 		)
-		(property "Footprint" "Switch_Keyboard_Hotswap_Kailh:SW_Hotswap_Kailh_MX_2.25u"
+		(property "Footprint" "Switch_Keyboard_Hotswap_Kailh:SW_Hotswap_Kailh_MX_1.50u"
 			(at 377.19 147.32 0)
 			(effects
@@
 	(symbol
 		(lib_id "Switch:SW_Push")
-		(at 351.79 180.34 180)
+		(at 351.79 180.34 0)
+		(mirror x)
 		(unit 1)
 		(exclude_from_sim no)
@@
 		(dnp no)
 		(property "Reference" "SW4_13"
-			(at 356.87 183.642 0)
+			(at 356.87 183.388 0)
 			(effects
 				(font
@@
 	(symbol
 		(lib_id "Switch:SW_Push")
-		(at 330.2 223.52 180)
+		(at 330.2 223.52 0)
+		(mirror x)
 		(unit 1)
 		(exclude_from_sim no)
@@
 		(dnp no)
 		(property "Reference" "SW5_13"
-			(at 323.596 225.552 0)
+			(at 323.342 225.552 0)
 			(effects
 				(font
@@
 			)
 		)
-		(property "Footprint" "Switch_Keyboard_Hotswap_Kailh:SW_Hotswap_Kailh_MX_1.25u"
+		(property "Footprint" "Switch_Keyboard_Hotswap_Kailh:SW_Hotswap_Kailh_MX_1.50u"
 			(at 330.2 228.6 0)
 			(effects
@@
 	(symbol
 		(lib_id "Switch:SW_Push")
-		(at 49.53 228.6 180)
+		(at 49.53 228.6 0)
+		(mirror x)
 		(unit 1)
 		(exclude_from_sim no)
@@
 		(dnp no)
 		(property "Reference" "SW5_4"
-			(at 45.212 231.648 0)
+			(at 44.958 231.648 0)
 			(effects
 				(font
@@
 			)
 		)
-		(property "Footprint" "Switch_Keyboard_Hotswap_Kailh:SW_Hotswap_Kailh_MX_1.25u"
+		(property "Footprint" "Switch_Keyboard_Hotswap_Kailh:SW_Hotswap_Kailh_MX_1.50u"
 			(at 49.53 233.68 0)
 			(effects
@@
 	(symbol
 		(lib_id "Switch:SW_Push")
-		(at 199.39 231.14 180)
+		(at 199.39 231.14 0)
+		(mirror x)
 		(unit 1)
 		(exclude_from_sim no)
@@
 		(dnp no)
 		(property "Reference" "SW5_9"
-			(at 203.962 234.442 0)
+			(at 203.454 233.934 0)
 			(effects
 				(font
@@
 			)
 		)
-		(property "Footprint" "Switch_Keyboard_Hotswap_Kailh:SW_Hotswap_Kailh_MX_6.25u"
+		(property "Footprint" "Switch_Keyboard_Hotswap_Kailh:SW_Hotswap_Kailh_MX_6.00u"
 			(at 199.39 236.22 0)
 			(effects
@@
 			)
 		)
-		(property "Footprint" "Switch_Keyboard_Hotswap_Kailh:SW_Hotswap_Kailh_MX_2.75u"
+		(property "Footprint" "Switch_Keyboard_Hotswap_Kailh:SW_Hotswap_Kailh_MX_1.00u"
 			(at 377.19 185.42 0)
 			(effects
@@
 	(symbol
 		(lib_id "Switch:SW_Push")
-		(at 378.46 66.04 180)
+		(at 378.46 66.04 0)
 		(unit 1)
 		(exclude_from_sim no)
@@
 		(dnp no)
 		(property "Reference" "SW1_14"
-			(at 374.142 69.088 0)
+			(at 378.46 68.072 0)
 			(effects
 				(font
@@
 		)
 		(property "Value" "SW_Push"
-			(at 378.46 71.12 0)
+			(at 378.46 60.96 0)
 			(effects
 				(font
@@
 		)
 		(property "Footprint" "Switch_Keyboard_Hotswap_Kailh:SW_Hotswap_Kailh_MX_2.00u"
-			(at 378.46 71.12 0)
+			(at 378.46 60.96 0)
 			(effects
 				(font
@@
 		)
 		(property "Datasheet" "~"
-			(at 378.46 71.12 0)
+			(at 378.46 60.96 0)
 			(effects
 				(font
@@
 	(symbol
 		(lib_id "Switch:SW_Push")
-		(at 354.33 227.33 180)
+		(at 354.33 227.33 0)
+		(mirror x)
 		(unit 1)
 		(exclude_from_sim no)
@@
 			)
 		)
-		(property "Footprint" "Switch_Keyboard_Hotswap_Kailh:SW_Hotswap_Kailh_MX_1.25u"
+		(property "Footprint" "Switch_Keyboard_Hotswap_Kailh:SW_Hotswap_Kailh_MX_1.00u"
 			(at 354.33 232.41 0)
 			(effects
@@
 	(symbol
 		(lib_id "Switch:SW_Push")
-		(at 303.53 227.33 180)
+		(at 303.53 227.33 0)
+		(mirror x)
 		(unit 1)
 		(exclude_from_sim no)
@@
 			)
 		)
-		(property "Footprint" "Switch_Keyboard_Hotswap_Kailh:SW_Hotswap_Kailh_MX_1.25u"
+		(property "Footprint" "Switch_Keyboard_Hotswap_Kailh:SW_Hotswap_Kailh_MX_1.50u"
 			(at 303.53 232.41 0)
 			(effects
@@
 			)
 		)
-		(property "Footprint" "Switch_Keyboard_Hotswap_Kailh:SW_Hotswap_Kailh_MX_2.00u"
+		(property "Footprint" "Switch_Keyboard_Hotswap_Kailh:SW_Hotswap_Kailh_MX_1.00u"
 			(at 378.46 78.74 0)
 			(effects
@@
 	(symbol
 		(lib_id "Switch:SW_Push")
-		(at 99.06 228.6 180)
+		(at 99.06 228.6 0)
+		(mirror x)
 		(unit 1)
 		(exclude_from_sim no)
@@
 			)
 		)
-		(property "Footprint" "Switch_Keyboard_Hotswap_Kailh:SW_Hotswap_Kailh_MX_1.25u"
+		(property "Footprint" "Switch_Keyboard_Hotswap_Kailh:SW_Hotswap_Kailh_MX_1.50u"
 			(at 99.06 233.68 0)
 			(effects
@@
 			)
 		)
-		(property "Footprint" "Switch_Keyboard_Hotswap_Kailh:SW_Hotswap_Kailh_MX_2.75u"
+		(property "Footprint" "Switch_Keyboard_Hotswap_Kailh:SW_Hotswap_Kailh_MX_1.75u"
 			(at 351.79 193.04 0)
 			(effects
@@
 	(symbol
 		(lib_id "Switch:SW_Push")
-		(at 73.66 228.6 180)
+		(at 73.66 228.6 0)
+		(mirror x)
 		(unit 1)
 		(exclude_from_sim no)
@@
 		(dnp no)
 		(property "Reference" "SW5_5"
-			(at 69.342 231.648 0)
+			(at 69.85 231.902 0)
 			(effects
 				(font
@@
 			)
 		)
-		(property "Footprint" "Switch_Keyboard_Hotswap_Kailh:SW_Hotswap_Kailh_MX_1.25u"
+		(property "Footprint" "Switch_Keyboard_Hotswap_Kailh:SW_Hotswap_Kailh_MX_1.00u"
 			(at 73.66 233.68 0)
 			(effects
@@
 	(symbol
 		(lib_id "Switch:SW_Push")
-		(at 199.39 223.52 180)
+		(at 199.39 223.52 0)
+		(mirror x)
 		(unit 1)
 		(exclude_from_sim no)
@@
 		(dnp no)
 		(property "Reference" "SW5_8"
-			(at 203.708 226.314 0)
+			(at 203.2 226.314 0)
 			(effects
 				(font
@@
 			)
 		)
-		(property "Footprint" "Switch_Keyboard_Hotswap_Kailh:SW_Hotswap_Kailh_MX_6.25u"
+		(property "Footprint" "Switch_Keyboard_Hotswap_Kailh:SW_Hotswap_Kailh_MX_7.00u"
 			(at 199.39 228.6 0)
 			(effects
@@
 	(symbol
 		(lib_id "Switch:SW_Push")
-		(at 379.73 227.33 180)
+		(at 379.73 227.33 0)
+		(mirror x)
 		(unit 1)
 		(exclude_from_sim no)
@@
 		(dnp no)
 		(property "Reference" "SW5_18"
-			(at 374.396 230.378 0)
+			(at 374.142 230.886 0)
 			(effects
 				(font
@@
 			)
 		)
-		(property "Footprint" "Switch_Keyboard_Hotswap_Kailh:SW_Hotswap_Kailh_MX_1.25u"
+		(property "Footprint" "Switch_Keyboard_Hotswap_Kailh:SW_Hotswap_Kailh_MX_1.50u"
 			(at 379.73 232.41 0)
 			(effects
@@
 					(unit 1)
 				)
-			)
-		)
-	)
-	(symbol
-		(lib_id "Switch:SW_Push")
-		(at 374.65 111.76 180)
-		(unit 1)
-		(exclude_from_sim no)
-		(in_bom yes)
-		(on_board yes)
-		(dnp no)
-		(property "Reference" "SW2_15"
-			(at 380.238 114.808 0)
-			(effects
-				(font
-					(size 1.27 1.27)
-				)
-			)
-		)
-		(property "Value" "SW_Push"
-			(at 374.65 116.84 0)
-			(effects
-				(font
-					(size 1.27 1.27)
-				)
-				(hide yes)
-			)
-		)
-		(property "Footprint" "Switch_Keyboard_Hotswap_Kailh:SW_Hotswap_Kailh_MX_1.50u"
-			(at 374.65 116.84 0)
-			(effects
-				(font
-					(size 1.27 1.27)
-				)
-				(hide yes)
-			)
-		)
-		(property "Datasheet" "~"
-			(at 374.65 116.84 0)
-			(effects
-				(font
-					(size 1.27 1.27)
-				)
-				(hide yes)
-			)
-		)
-		(property "Description" ""
-			(at 374.65 111.76 0)
-			(effects
-				(font
-					(size 1.27 1.27)
-				)
-			)
-		)
-		(pin "1"
-		)
-		(pin "2"
-		)
-		(instances
-			(project "goose60rev2"
-				(path "/6ebc9a41-9721-4591-a32f-d06e561fa915/7b305d81-944e-47f6-9e16-05645e53394c"
-					(reference "SW2_15")
-					(unit 1)
-				)

Commit message: [WIP] update PCB layout
Other:
- note added: "2025.11.12"
- note added: "keyboard matrix"
- note added: "rev2"
Changed lines of the file:
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@@
+		)
+	)
+	(text "keyboard matrix"
+		(exclude_from_sim no)
+		(at 321.818 261.366 0)
+		(effects
+			(font
+				(size 2.54 2.54)
+				(thickness 0.508)
+				(bold yes)
+			)
 		)
 	)
@@
 		)
 	)
+	(text "2025.11.12"
+		(exclude_from_sim no)
+		(at 335.534 280.416 0)
+		(effects
+			(font
+				(size 1.27 1.27)
+				(thickness 0.508)
+				(bold yes)
+			)
+		)
+	)
 	(text "]"
 		(exclude_from_sim no)
@@
 		)
 	)
+	(text "keyboard matrix"
+		(exclude_from_sim no)
+		(at 320.294 276.606 0)
+		(effects
+			(font
+				(size 1.778 1.778)
+				(thickness 0.508)
+				(bold yes)
+			)
+		)
+	)
 	(text "\\\nBS [HHKB]"
 		(exclude_from_sim no)
@@
 		)
 	)
+	(text "rev2"
+		(exclude_from_sim no)
+		(at 394.716 280.162 0)
+		(effects
+			(font
+				(size 1.27 1.27)
+				(thickness 0.508)
+				(bold yes)
+			)
+		)
+	)

Commit message: add stabilizer and remove 6u hhkb support
Parts:
- removed SW5_14: SW_Push, Switch_Keyboard_Hotswap_Kailh:SW_Hotswap_Kailh_MX_1.00u, symbol Switch:SW_Push
- removed SW5_9: SW_Push, Switch_Keyboard_Hotswap_Kailh:SW_Hotswap_Kailh_MX_6.00u, symbol Switch:SW_Push
Changed lines of the file:
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@@
 	)
 	(junction
-		(at 191.77 223.52)
-		(diameter 0)
-		(color 0 0 0 0)
-	)
-	(junction
 		(at 82.55 228.6)
 		(diameter 0)
@@
 	)
 	(junction
-		(at 318.77 223.52)
-		(diameter 0)
-		(color 0 0 0 0)
-	)
-	(junction
 		(at 233.68 91.44)
 		(diameter 0)
@@
 	)
 	(junction
-		(at 336.55 229.87)
-		(diameter 0)
-		(color 0 0 0 0)
-	)
-	(junction
 		(at 59.69 69.85)
 		(diameter 0)
@@
 	)
 	(junction
-		(at 209.55 231.14)
-		(diameter 0)
-		(color 0 0 0 0)
-	)
-	(junction
 		(at 389.89 73.66)
 		(diameter 0)
@@
 	(wire
 		(pts
-			(xy 191.77 223.52) (xy 191.77 231.14)
-		)
-		(stroke
-			(width 0)
-			(type default)
-		)
-	)
-	(wire
-		(pts
 			(xy 335.28 129.54) (xy 335.28 135.89)
 		)
@@
 	(wire
 		(pts
-			(xy 318.77 223.52) (xy 318.77 229.87)
-		)
-		(stroke
-			(width 0)
-			(type default)
-		)
-	)
-	(wire
-		(pts
 			(xy 121.92 173.99) (xy 121.92 184.15)
 		)
@@
 	(wire
 		(pts
-			(xy 194.31 231.14) (xy 191.77 231.14)
-		)
-		(stroke
-			(width 0)
-			(type default)
-		)
-	)
-	(wire
-		(pts
 			(xy 158.75 107.95) (xy 161.29 107.95)
 		)
@@
 	(wire
 		(pts
-			(xy 320.04 229.87) (xy 318.77 229.87)
-		)
-		(stroke
-			(width 0)
-			(type default)
-		)
-	)
-	(wire
-		(pts
 			(xy 344.17 142.24) (xy 346.71 142.24)
 		)
@@
 	(wire
 		(pts
-			(xy 330.2 229.87) (xy 336.55 229.87)
-		)
-		(stroke
-			(width 0)
-			(type default)
-		)
-	)
-	(wire
-		(pts
 			(xy 356.87 187.96) (xy 361.95 187.96)
 		)
@@
 	(wire
 		(pts
-			(xy 204.47 231.14) (xy 209.55 231.14)
-		)
-		(stroke
-			(width 0)
-			(type default)
-		)
-	)
-	(wire
-		(pts
 			(xy 78.74 228.6) (xy 82.55 228.6)
 		)
@@
 	)
 	(symbol
-		(lib_id "Switch:SW_Push")
-		(at 325.12 229.87 180)
-		(unit 1)
-		(exclude_from_sim no)
-		(in_bom yes)
-		(on_board yes)
-		(dnp no)
-		(property "Reference" "SW5_14"
-			(at 332.486 231.902 0)
-			(effects
-				(font
-					(size 1.27 1.27)
-				)
-			)
-		)
-		(property "Value" "SW_Push"
-			(at 325.12 234.95 0)
-			(effects
-				(font
-					(size 1.27 1.27)
-				)
-				(hide yes)
-			)
-		)
-		(property "Footprint" "Switch_Keyboard_Hotswap_Kailh:SW_Hotswap_Kailh_MX_1.00u"
-			(at 325.12 234.95 0)
-			(effects
-				(font
-					(size 1.27 1.27)
-				)
-				(hide yes)
-			)
-		)
-		(property "Datasheet" "~"
-			(at 325.12 234.95 0)
-			(effects
-				(font
-					(size 1.27 1.27)
-				)
-				(hide yes)
-			)
-		)
-		(property "Description" ""
-			(at 325.12 229.87 0)
-			(effects
-				(font
-					(size 1.27 1.27)
-				)
-			)
-		)
-		(pin "1"
-		)
-		(pin "2"
-		)
-		(instances
-			(project "goose60rev2"
-				(path "/6ebc9a41-9721-4591-a32f-d06e561fa915/7b305d81-944e-47f6-9e16-05645e53394c"
-					(reference "SW5_14")
-					(unit 1)
-				)
-			)
-		)
-	)
-	(symbol
 		(lib_id "Diode:1N4148")
 		(at 280.67 59.69 180)
@@
 					(unit 1)
 				)
-			)
-		)
-	)
-	(symbol
-		(lib_id "Switch:SW_Push")
-		(at 199.39 231.14 0)
-		(mirror x)
-		(unit 1)
-		(exclude_from_sim no)
-		(in_bom yes)
-		(on_board yes)
-		(dnp no)
-		(property "Reference" "SW5_9"
-			(at 203.454 233.934 0)
-			(effects
-				(font
-					(size 1.27 1.27)
-				)
-			)
-		)
-		(property "Value" "SW_Push"
-			(at 199.39 236.22 0)
-			(effects
-				(font
-					(size 1.27 1.27)
-				)
-				(hide yes)
-			)
-		)
-		(property "Footprint" "Switch_Keyboard_Hotswap_Kailh:SW_Hotswap_Kailh_MX_6.00u"
-			(at 199.39 236.22 0)
-			(effects
-				(font
-					(size 1.27 1.27)
-				)
-				(hide yes)
-			)
-		)
-		(property "Datasheet" "~"
-			(at 199.39 236.22 0)
-			(effects
-				(font
-					(size 1.27 1.27)
-				)
-				(hide yes)
-			)
-		)
-		(property "Description" ""
-			(at 199.39 231.14 0)
-			(effects
-				(font
-					(size 1.27 1.27)
-				)
-			)
-		)
-		(pin "1"
-		)
-		(pin "2"
-		)
-		(instances
-			(project "goose60rev2"
-				(path "/6ebc9a41-9721-4591-a32f-d06e561fa915/7b305d81-944e-47f6-9e16-05645e53394c"
-					(reference "SW5_9")
-					(unit 1)
-				)
